Commit message: feat: sim improvements, Docker fixes, repo cleanup
- Add side + RGB cameras to robot model (tb.sdf.xacro)
- Add sim_only_launch.py, square_room world, ArUco marker 42 model
- Add macOS Docker Compose + devcontainer + FastDDS configs
- Fix DDS communication (remove restrictive FASTRTPS profile)
- Fix TURTLEBOT3_MODEL default: burger → waffle
- Decouple g3gzsim from g3g_frontier_exploration (package.xml)
- Gitignore local dev tools (sim_dashboard, scripts, DDS fix dirs)

File: src/g3gzsim/urdf/tb.sdf.xacro (robot description, xacro)
@@ -378,4 +378,23 @@
           </camera>
         </sensor>
+        <sensor name="rgb_camera" type="camera">
+          <always_on>1</always_on>
+          <update_rate>30</update_rate>
+          <pose>0.064 -0.047 0.107 0 0 0</pose>
+          <topic>$(arg namespace)/camera/image_raw</topic>
+          <gz_frame_id>camera_rgb_optical_frame</gz_frame_id>
+          <camera name="rgb_camera">
+            <horizontal_fov>1.047</horizontal_fov>
+            <image>
+              <width>640</width>
+              <height>480</height>
+              <format>R8G8B8</format>
+            </image>
+            <clip>
+              <near>0.1</near>
+              <far>100.0</far>
+            </clip>
+          </camera>
+        </sensor>
       </link>
       <joint name="base_joint" type="fixed">
@@ -423,4 +442,39 @@
           <xyz>0 0 1</xyz>
         </axis>
+      </joint>
+      <!-- Side camera: right side of robot, pointing -Y (starboard) -->
+      <link name="side_camera_link">
+        <inertial>
+          <pose>0.0 -0.132 0.107 0 0 -1.5708</pose>
+          <inertia>
+            <ixx>0.001</ixx> <ixy>0</ixy> <ixz>0</ixz>
+            <iyy>0.001</iyy> <iyz>0</iyz> <izz>0.001</izz>
+          </inertia>
+          <mass>0.035</mass>
+        </inertial>
+        <pose>0.0 -0.132 0.107 0 0 -1.5708</pose>
+        <sensor name="side_rgb_camera" type="camera">
+          <always_on>1</always_on>
+          <update_rate>30</update_rate>
+          <pose>0.0 -0.132 0.107 0 0 -1.5708</pose>
+          <topic>$(arg namespace)/side_camera/image_raw</topic>
+          <gz_frame_id>side_camera_optical_frame</gz_frame_id>
+          <camera name="side_rgb_camera">
+            <horizontal_fov>1.047</horizontal_fov>
+            <image>
+              <width>640</width>
+              <height>480</height>
+              <format>R8G8B8</format>
+            </image>
+            <clip>
+              <near>0.1</near>
+              <far>100.0</far>
+            </clip>
+          </camera>
+        </sensor>
+      </link>
+      <joint name="side_camera_joint" type="fixed">
+        <parent>base_link</parent>
+        <child>side_camera_link</child>
       </joint>
       <plugin
